File: PCB/WP-2_IC_Card_RAM_128K_v2_bare.kicad_pcb (KiCad board)
At the start: 2 copper layers, 45 x 54 mm, 4 parts, among them J1 Conn_01x38_Female, U1 SRAM 128Kx8 5v Parallel, U2 SRAM 128Kx8 5v Parallel

Commit message: simple version
Parts:
- J1: footprint 0_LOCAL:PinSocket_1x38x1.27_edge_ext -> 0_LOCAL:PinSocket_1x38x1.27_edge_s
Routing:
- net /A9: track 18.1 -> 16.9 mm
Other:
- outline, holes or cut-outs redrawn
- board text removed: "Socket header 4.4mm"
