File: PCB/WP-2_IC_Card_RAM_128K_bare.kicad_pcb (KiCad board)
At the start: 2 copper layers, 45 x 54 mm, 10 parts, among them J1 Conn_01x38_Female, U1 SRAM 128Kx8 5v Parallel, U2 SRAM 128Kx8 5v Parallel

Commit message: v003
Parts:
- removed D1: 1N4148, Diodes_SMD:D_0805
- removed the R2 at (153.0, 119.4)
- removed R3: 47K, Resistors_SMD:R_0805
- C1: value 470+uf -> 220uf; footprint Capacitors_SMD:C_0805 -> 0_LOCAL:CP_Tantalum_Case-B_EIA-3528-21_Reflow
- R1: value 500 -> 4.7K; footprint Resistors_SMD:R_0805 -> 0_LOCAL:R_0805
- R2: renamed from R4; footprint Resistors_SMD:R_0805 -> 0_LOCAL:R_0805
- moved R1 7.11 mm to (150.8, 112.2), turned to 270 degrees
- moved C1 2.36 mm to (151.5, 116.7), turned to 270 degrees
- moved U1 0.75 mm to (149.2, 99.7)
- moved U2 0.75 mm to (149.2, 99.7)
Connections:
- R1 pad 1: VMEM -> VDD
- U1 pad 8: VMEM -> VDD
- U2 pad 8: VMEM -> VDD
Routing:
- net VMEM: track 48.9 -> 0.00 mm, vias 2 -> 0
- net VDD: track 3.84 -> 24.4 mm
- net GND: track 77.8 -> 68.6 mm
- net /R~W: track 21.2 -> 20.2 mm
- net /A9: track 15.2 -> 14.4 mm
- net /CE2: track 40.6 -> 39.8 mm
- net /~CE1: track 21.2 -> 20.4 mm, vias 3 -> 2
- net /D7: track 13.9 -> 13.2 mm
- net /D6: track 13.6 -> 12.9 mm
- net /D5: track 13.9 -> 13.2 mm
- net /D4: track 14.7 -> 14.0 mm
- net /D3: track 15.8 -> 15.1 mm
- net /D2: track 15.6 -> 14.8 mm
- net /D0: track 17.1 -> 16.3 mm
- net /A8: track 14.5 -> 13.8 mm
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Other:
- board text added: "bare_003"
- board text removed: "bare_002"
