File: PCB/WP-2_IC_Card_RAM_128K_003.kicad_pcb (KiCad board)
At the start: 2 copper layers, 14.5 x 48.5 mm, 9 parts, among them J1 Conn_01x38_Female, U1 SRAM 128Kx8 5v Parallel, U2 SRAM 128Kx8 5v Parallel

Commit message: v002, v003
Parts:
- removed REF** (x2): npth_3mm, 0_LOCAL:npth_3mm
- added Carrier: Carrier_v003, 0_LOCAL:Carrier_v003, F.Cu at (158.8, 99.7)
Other:
- board text added: "v003"
- board text removed: "003"
