File: PCB/WP-2_IC_Card_ROM.kicad_pcb (KiCad board)
At the start: 2 copper layers, 45 x 54 mm, 5 parts, among them J1 Conn_01x38_Female, U1 FLASH 256Kx8 5v Parallel, U2 FLASH 256Kx8 5v Parallel

Commit message: kicad 6
Connections:
- net /R~W renamed /R~{W}
- net /~CE1 renamed /~{CE1}
- net /~OE renamed /~{OE}
- net /~WE renamed /~{WE}
Routing:
- net GND: track 29.4 -> 0.00 mm, vias 3 -> 5
- added copper zone on B.Cu, net GND
- added copper zone on F.Cu, net GND
Other:
- net class Default removed
- board text added: "PCB thickness 1.2mm"
- board text added: "WP-2_IC_Card_ROM v004"
- board text removed: "WP-2_IC_Card_ROM v003"
