File: PCB/WP-2_IC-Card_MRAM_512K.kicad_sch (KiCad schematic)
At the start: 25 parts, among them J1 SMS-138-01-G-S, SW1 CUS-14TB, U1 MR2A08xxYSxxx, U2 MIC5317-3.3YD5, U3 4245, U4 4245, U5 4245, U6 4245

Commit message: file names, page titles, mram relocate parts
Other:
- title: WP-2_IC-Card_MRAM_512 -> WP-2_IC-Card_MRAM_512K
Changed lines of the file:
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@@
 	(paper "USLetter")
 	(title_block
-		(title "WP-2_IC-Card_MRAM_512")
-		(date "2023-12-09")
-		(rev "014")
+		(title "WP-2_IC-Card_MRAM_512K")
+		(date "2024-08-22")
+		(rev "015")
 		(company "Brian K. White - b.kenyon.w@gmail.com")
 	)
