File: PCB/WP-2_IC-Card_ROM_thin_switch.kicad_pcb (KiCad board)
At the start: 2 copper layers, 54 x 54 mm, 11 parts, among them J1 SMS-138-01-G-S, SW1 Write-Enable, U1 29F0x0_TSOP

Commit message: ram & rom boms
Parts:
- SW1: footprint 000_LOCAL:CUS-12TB pth -> 000_LOCAL:SW3_JS102000SAQN_CNK
Routing:
- net /~{WE}: track 7.95 -> 7.27 mm
