File: PCB/WP-2_IC-Card_Programming_Adapter_virt.kicad_sch (KiCad schematic)
At the start: 3 parts, among them J1 TMS-138-01, J2 SST39SF020_DIP, J3 Conn_02x08_Odd_Even

Commit message: silkscreen, remove old 128k sram, new programming adapter
Other:
- title: TANDY WP-2 IC Card Programming Adapter -> TANDY WP-2 IC Card Programming Adapter virt
